File: panelolu 2.1.brd (EAGLE design)
At the start: 98 x 25 mm, 24 parts, among them IC1 LM340MP-05, IC2 4050D, IC3 MCP23017SO28, SW1 EC12E_SW

Commit message: Update panelolu 2.1.brd
Change voltage regulator MIC5209-3.3YS
Parts:
- IC1: value LM340MP-05 -> MIC5209-3.3YS
Changed lines of the file:
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@@
 <?xml version="1.0" encoding="utf-8"?>
 <!DOCTYPE eagle SYSTEM "eagle.dtd">
-<eagle version="6.2">
+<eagle version="6.4">
 <drawing>
 <settings>
@@
 </class>
 </classes>
-<designrules>
+<designrules name="default">
 <description language="de">&lt;b&gt;EAGLE Design Rules&lt;/b&gt;
 &lt;p&gt;
@@
 <attribute name="OC_NEWARK" value="74M1068" x="60.96" y="10.16" size="1.778" layer="27" rot="R270.1" display="off"/>
 </element>
-<element name="IC1" library="linear" package="SOT223" value="LM340MP-05" x="74.068" y="4.326" smashed="yes" rot="MR90">
+<element name="IC1" library="linear" package="SOT223" value="MIC5209-3.3YS" x="74.068" y="4.326" smashed="yes" rot="MR90">
 <attribute name="NAME" x="74.1188" y="1.786" size="1.27" layer="26" rot="MR90"/>
 </element>
